File: hardware/schematics/phasedriver.kicad_sch (KiCad schematic)
At the start: 6 parts, among them Q1 30N06_C5807887, Q2 30N06_C5807887, U3 SLM2003ECA-DG

Commit message: Arrange components
Parts:
- added C16, C17, C18: 100n, Capacitor_SMD:C_0603_1608Metric, symbol Device:C
- added C19: RVT1J221M1010, easyeda2kicad:CAP-SMD_BD10.0-L10.3-W10.3-FD, symbol easyeda2kicad:RVT1J221M1010
- added D1: SS14_C2837270, easyeda2kicad:SMA_L4.3-W2.6-LS5.0-RD, symbol easyeda2kicad:SS14_C2837270
- added TP1: TestPoint, TestPoint:TestPoint_Pad_4.0x4.0mm, symbol Connector:TestPoint
- added U4: INA180A3IDBVR, easyeda2kicad:SOT-23-5_L3.0-W1.7-P0.95-LS2.8-BR, symbol easyeda2kicad:INA180A3IDBVR
Connections:
- net +12V: now also C16.1, D1.2 (A); no longer U3.8 (VB)
- net GND: now also C18.2, C19.2, U4.2 (GND), U4.4 (IN-); no longer U3.4 (COM)
- net VCC: now also C19.1
- net at Q2.3 (S), R10.1: now also U3.4 (COM), C16.2, U4.3 (IN+)
- net phase: no longer names the net of Q1.3 (S), Q2.2 (D), U3.6 (VS)
- net phase: now also C17.2, TP1.1
- new net: C17.1, D1.1 (C), U3.8 (VB)
- new net 5V: C18.1, U4.5 (V+)
- new net AOUT: U4.1 (OUT)

Commit message: Add more routing
Connections:
- net 5V renamed +3V3
Changed lines of the file:
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@@
 		)
 	)
-	(hierarchical_label "5V"
+	(hierarchical_label "+3V3"
 		(shape input)
 		(at 76.2 106.68 180)
